File: PCB design/self_balancing_robot.kicad_pcb (KiCad board)
At the start: 2 copper layers, 29 parts, among them J1 I2C, J2 Conn_01x06_Socket, J3 Conn_01x02_Socket, J4 Conn_01x04_Socket, J6 SPI, J7 Conn_01x04_Pin, SW1 SW_Push, U1 ATmega328P-A, U2 L293D, U4 LP2985-3.3, U5 NCP1117-5.0_SOT223, Y1 Crystal

Commit message: PCB update - almost finishing
Parts:
- removed U2: L293D, Package_DIP:DIP-16_W7.62mm
- added J5: L293D_left, Connector_PinSocket_2.54mm:PinSocket_1x08_P2.54mm_Vertical, F.Cu at (136.5, 88.7)
- added J8: L293D_right, Connector_PinSocket_2.54mm:PinSocket_1x08_P2.54mm_Vertical, F.Cu at (144.5, 88.8)
- added J9: input_supply, Connector_TE-Connectivity:TE_826576-2_1x02_P3.96mm_Vertical, F.Cu at (87.3, 115.0)
- C1, C12, C13, C14, C2, C3, C4, C5, C6, C7, C8: footprint Capacitor_THT:C_Disc_D5.0mm_W2.5mm_P2.50mm -> Capacitor_SMD:C_0805_2012Metric
- D1: footprint Resistor_THT:R_Axial_DIN0204_L3.6mm_D1.6mm_P5.08mm_Horizontal -> Resistor_THT:R_Axial_DIN0207_L6.3mm_D2.5mm_P7.62mm_Horizontal
- J2: value Conn_01x06_Socket -> Analog
- J3: value Conn_01x02_Socket -> left_engine; footprint Connector_PinSocket_2.54mm:PinSocket_1x02_P2.54mm_Vertical -> Connector_TE-Connectivity:TE_826576-2_1x02_P3.96mm_Vertical
- J4: value Conn_01x04_Socket -> right_engine; footprint Connector_PinSocket_2.54mm:PinSocket_1x04_P2.54mm_Vertical -> Connector_TE-Connectivity:TE_826576-2_1x02_P3.96mm_Vertical
- J7: value Conn_01x04_Pin -> UART
- moved J6 123.6 mm to (63.9, 101.8), turned to -90 degrees
- moved Y1 87.2 mm to (68.0, 92.5)
- moved C7 86.6 mm to (73.7, 88.2), turned to 180 degrees
- moved J7 82.3 mm to (95.1, 77.5), turned to 90 degrees
- moved U4 76.8 mm to (123.0, 93.2)
- moved J1 73.9 mm to (118.9, 88.2), turned to 90 degrees
- moved U1 69.4 mm to (100.8, 88.5)
- moved J4 56.3 mm to (127.5, 115.5)
- moved C6 52.0 mm to (67.0, 88.2)
- moved J2 52.0 mm to (130.6, 72.0), turned to -90 degrees
- moved C12 46.3 mm to (96.2, 106.5), turned to -90 degrees
- moved SW1 42.8 mm to (110.2, 82.8)
- moved C13 40.4 mm to (96.2, 102.8), turned to -90 degrees
- moved R1 39.7 mm to (110.2, 77.5), turned to -90 degrees
- moved C1 36.2 mm to (91.4, 86.2), turned to 180 degrees
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Connections:
- J3 pad 1: GND -> ENGINE_LEFT_GND
- J3 pad 2: Net-(D1-A) -> ENGINE_LEFT_VCC
- J4 pad 1: ENGINE_LEFT_GND -> ENGINE_RIGHT_VCC
- J4 pad 2: ENGINE_LEFT_VCC -> ENGINE_RIGHT_GND
- R4 pad 1: +5V -> +3V3
- R5 pad 1: +5V -> +3V3
Routing:
- net +7.2V: track 0.00 -> 3.88 mm
Other:
- board outline added: 72.8 x 44.8 mm
