File: PCB design/self_balancing_robot.kicad_sch (KiCad schematic)
At the start: 28 parts, among them J1 Conn_01x05_Socket, J2 Conn_01x04_Socket, J3 Conn_01x02_Socket, J4 Conn_01x04_Socket, SW1 SW_Push, U1 ATmega328P-A, U2 L293D, U3 LM1117MP-3.3, U4 LM1117T-5.0, Y1 Crystal

Commit message: PCB update
Parts:
- removed J2: Conn_01x04_Socket, Connector_PinSocket_2.54mm:PinSocket_1x04_P2.54mm_Vertical, symbol Connector:Conn_01x04_Socket
- added D3: LED, symbol Device:LED
- added J5: Conn_01x07_Socket, symbol Connector:Conn_01x07_Socket
- added J6: SPI, symbol Connector:Conn_01x06_Socket
- added J7: Conn_01x04_Pin, symbol Connector:Conn_01x04_Pin
- added R3: 330, symbol Device:R_Small
Connections:
- net +5V: now also J6.1 (Pin_1), J7.4 (Pin_4)
- net GND: now also D3.1 (K), J6.2 (Pin_2), J7.1 (Pin_1)
- net RX_CONN: now also J7.3 (Pin_3)
- net TX_CONN: now also J7.2 (Pin_2)
- net PD6: now reaches U1.10 (PD6)
- net PD6: now also J5.7 (Pin_7)
- net CS: now reaches U1.14 (PB2)
- net CS: now also J6.6 (Pin_6)
- net MOSI: now reaches U1.15 (PB3)
- net MOSI: now also J6.4 (Pin_4)
- net MISO: now reaches U1.16 (PB4)
- net MISO: now also J6.3 (Pin_3)
- net SCK: now reaches U1.17 (PB5)
- net SCK: now also J6.5 (Pin_5), R3.1
- net A6: now reaches U1.19 (ADC6)
- net A6: now also J5.5 (Pin_5)
- net A7: now reaches U1.22 (ADC7)
- net A7: now also J5.6 (Pin_6)
- net A0: now reaches U1.23 (PC0)
- net A0: now also J5.1 (Pin_1)
- net A1: now reaches U1.24 (PC1)
- net A1: now also J5.2 (Pin_2)
- net A2: now reaches U1.25 (PC2)
- net A2: now also J5.3 (Pin_3)
- net A3: now reaches U1.26 (PC3)
- net A3: now also J5.4 (Pin_4)
- new net: D3.2 (A), R3.2
- no-connect marks 11 -> 0
Other:
- moved on the sheet: C6, C7, C8, R1, SW1, Y1

Commit message: PCB update
Parts:
- removed C10, C11: 100nF, Capacitor_THT:C_Disc_D5.0mm_W2.5mm_P2.50mm, symbol Device:C_Small
- removed C9: 10uF, Capacitor_THT:CP_Radial_D5.0mm_P2.50mm, symbol Device:C_Polarized
- removed D1: 1N4007, Diode_THT:D_DO-41_SOD81_P10.16mm_Horizontal, symbol Diode:1N4007
- removed D2: LED, Capacitor_THT:CP_Radial_D5.0mm_P2.50mm, symbol Device:LED
- removed J5: Conn_01x07_Socket, symbol Connector:Conn_01x07_Socket
- removed R2: 220R, symbol Device:R
- removed U3: LM1117MP-3.3, Package_TO_SOT_SMD:SOT-223-3_TabPin2, symbol Regulator_Linear:LM1117MP-3.3
- removed U4: LM1117T-5.0, Package_TO_SOT_THT:TO-220-3_Vertical, symbol Regulator_Linear:LM1117T-5.0
- removed Y1: Crystal, symbol Device:Crystal_GND24
- added D1: D_Schottky, Resistor_THT:R_Axial_DIN0204_L3.6mm_D1.6mm_P5.08mm_Horizontal, symbol Device:D_Schottky
- added J2: Conn_01x06_Socket, Connector_PinSocket_2.54mm:PinSocket_1x06_P2.54mm_Vertical, symbol Connector:Conn_01x06_Socket
- added R4, R5: 4.7k, Resistor_SMD:R_0805_2012Metric, symbol Device:R
- added U4: LP2985-3.3, Package_TO_SOT_SMD:SOT-23-5, symbol Regulator_Linear:LP2985-3.3
- added U5: NCP1117-5.0_SOT223, Package_TO_SOT_SMD:SOT-223-3_TabPin2, symbol Regulator_Linear:NCP1117-5.0_SOT223
- added Y1: Crystal, Crystal:Crystal_HC49-4H_Vertical, symbol Device:Crystal
- C12, C13: value 100nF -> 47uF
- C5: value 100nF -> 1uF
- D3: footprint (none) -> LED_SMD:LED_1206_3216Metric
- J1: value Conn_01x05_Socket -> I2C
- J6: footprint (none) -> Connector_PinSocket_2.54mm:PinSocket_1x06_P2.54mm_Vertical
- J7: footprint (none) -> Connector_PinHeader_2.54mm:PinHeader_1x04_P2.54mm_Vertical
- R1, R3: footprint (none) -> Resistor_SMD:R_0805_2012Metric
Connections:
- net +7.2VA is gone; now on net +7.2V: C12.2, U2.8 (VCC2)
- net +3V3: now also U4.5 (VOUT)
- net +5V: now also R4.1, R5.1, U4.1 (VIN), U4.3 (ON/~{OFF}), U5.2 (VO)
- net +7.2V: now also D1.1 (K), U5.3 (VI); no longer J3.2 (Pin_2)
- net A0: now also J2.1 (Pin_1)
- net A1: now also J2.2 (Pin_2)
- net A2: now also J2.3 (Pin_3)
- net A3: now also J2.4 (Pin_4)
- net A6: now also J2.5 (Pin_5)
- net A7: now also J2.6 (Pin_6)
- net GND: now also U4.2 (GND), U4.4 (BP), U5.1 (GND)
- net PD6: now also R3.1
- net SCK: no longer R3.1
- net SCL_CONN: now also R4.2
- net SDA_CONN: now also R5.2
- net XTAL1_CONN: now also Y1.1
- net XTAL2_CONN: now also Y1.2
- new net: D1.2 (A), J3.2 (Pin_2)
Other:
- company: (none) -> Joanna Chrobot
- title: (none) -> Self Balancing robot
- moved on the sheet: C12, C13, C4, C5, J1, J3, J6

Commit message: PCB update - almost finishing
Parts:
- removed J3: Conn_01x02_Socket, Connector_PinSocket_2.54mm:PinSocket_1x02_P2.54mm_Vertical, symbol Connector:Conn_01x02_Socket
- removed J4: Conn_01x04_Socket, Connector_PinSocket_2.54mm:PinSocket_1x04_P2.54mm_Vertical, symbol Connector:Conn_01x04_Socket
- removed U2: L293D, Package_DIP:DIP-16_W7.62mm, symbol Driver_Motor:L293D
- added J3: left_engine, Connector_TE-Connectivity:TE_826576-2_1x02_P3.96mm_Vertical, symbol Connector:Screw_Terminal_01x02
- added J4: right_engine, Connector_TE-Connectivity:TE_826576-2_1x02_P3.96mm_Vertical, symbol Connector:Screw_Terminal_01x02
- added J5: L293D_left, Connector_PinSocket_2.54mm:PinSocket_1x08_P2.54mm_Vertical, symbol Connector:Conn_01x08_Socket
- added J8: L293D_right, Connector_PinSocket_2.54mm:PinSocket_1x08_P2.54mm_Vertical, symbol Connector:Conn_01x08_Socket
- added J9: input_supply, Connector_TE-Connectivity:TE_826576-2_1x02_P3.96mm_Vertical, symbol Connector:Screw_Terminal_01x02
- C1, C12, C13, C14, C2, C3, C4, C5, C6, C7, C8: footprint Capacitor_THT:C_Disc_D5.0mm_W2.5mm_P2.50mm -> Capacitor_SMD:C_0805_2012Metric
- D1: footprint Resistor_THT:R_Axial_DIN0204_L3.6mm_D1.6mm_P5.08mm_Horizontal -> Resistor_THT:R_Axial_DIN0207_L6.3mm_D2.5mm_P7.62mm_Horizontal
- J2: value Conn_01x06_Socket -> Analog
- J7: value Conn_01x04_Pin -> UART
Connections:
- net +3V3: now also R4.1, R5.1
- net +5V: now also J8.8 (Pin_8); no longer R4.1, R5.1
- net +7.2V: now also J5.8 (Pin_8)
- net ENGINE_LEFT_GND: now also J3.1 (Pin_1), J5.3 (Pin_3)
- net ENGINE_LEFT_VCC: now also J3.2 (Pin_2), J5.6 (Pin_6)
- net ENGINE_RIGHT_GND: now also J4.2 (Pin_2), J8.6 (Pin_6)
- net ENGINE_RIGHT_VCC: now also J4.1 (Pin_1), J8.3 (Pin_3)
- net GND: now also J5.4 (Pin_4), J5.5 (Pin_5), J8.4 (Pin_4), J8.5 (Pin_5), J9.1 (Pin_1)
- net PB0: now also J5.2 (Pin_2)
- net PB1: now also J5.1 (Pin_1)
- net PD3: now also J8.1 (Pin_1)
- net PD4: now also J8.7 (Pin_7)
- net PD5: now also J8.2 (Pin_2)
- net PD7: now also J5.7 (Pin_7)
- net at D1.2 (A): now also J9.2 (Pin_2)
